File: PCB/Mainboard/HonkLock.kicad_sch (KiCad schematic)
At the start: 10 parts, among them J1 Conn_01x03_Pin, J5 Conn_01x02_Pin, U2 ESP32-S3-SUPERMINI

Commit message: Mainboard ready for mfg
Parts:
- removed C2: 0.1uF, Capacitor_SMD:C_1206_3216Metric, symbol Device:C
- added C5: 0.1uF, Capacitor_SMD:C_0805_2012Metric, symbol Device:C
- added C6: 1uF, Capacitor_SMD:C_0805_2012Metric, symbol Device:C
- added R10, R8: 10k, Resistor_SMD:R_0805_2012Metric, symbol PCM_SparkFun-Resistor:R
- added R6, R7: 33k, Resistor_SMD:R_0805_2012Metric, symbol PCM_SparkFun-Resistor:R
- C1: footprint Capacitor_SMD:C_1206_3216Metric -> Capacitor_SMD:C_0805_2012Metric
- R2, R3: footprint Resistor_SMD:R_1206_3216Metric -> Resistor_SMD:R_0805_2012Metric
Connections:
- net 3v3: now also C5.1, C6.1, R10.1, R6.2, R7.1, R8.2
- net GND: now also C5.2, C6.2
- net BusSCL: now reaches RJ1.6
- net BusSCL: now also U1.7 (LY), R8.1; no longer U1.6 (SY)
- net BusSDA: now reaches RJ1.2
- net BusSDA: now also U1.2 (LX), R10.2; no longer U1.7 (LY)
- net Sensor1SCK renamed MCUSDA
- net MCUSDA: now also U1.3 (SX), R7.2; no longer U1.2 (LX)
- net Sensor1SDA renamed MCUSCL
- net MCUSCL: now also U1.6 (SY), R6.1; no longer U1.3 (SX)
- no-connect marks 18 -> 20
Other:
- note added: "Alternative to USB port"
- note added: "Cat5 should be 50pF/m"
- note added: "I2C Bus Extender"
- note added: "Power"
- note added: "USB-C that (should) work with A-C and C-C cables. Not USB-PD, just 5v1.5a"
- company: (none) -> tmuWolverine
- title: (none) -> HonkLock
- moved on the sheet: C1, J1, J5, R2, R3, U1, U2, USB1

Commit message: sent to mfg
Parts:
- J1: footprint Connector_JST:JST_XH_S3B-XH-A_1x03_P2.50mm_Horizontal -> Circuits_Connectors:CONN-TH_S3B-XH-A-LF-SN
- RJ1: footprint Circuits:RJ45-TH_HC-WK88-H16-DB -> Circuits_Connectors:RJ45-TH_HC-WK88-H16-DB
- U1: footprint EasyEDA_Lib:SOIC-8_L4.9-W3.9-P1.27-LS6.0-BL -> Circuits:SOIC-8_L4.9-W3.9-P1.27-LS6.0-BL
- U2: footprint Circuits:ESP32_S3_Supermini -> Circuits_MCU:ESP32_S3_Supermini
- USB1: footprint EasyEDA_Lib:USB-C-SMD_TYPE-C-16PIN-2MD-073 -> Circuits_Connectors:USB-C-SMD_TYPE-C-16PIN-2MD-073
Changed lines of the file:
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@@
 			)
 		)
-		(property "Footprint" "EasyEDA_Lib:SOIC-8_L4.9-W3.9-P1.27-LS6.0-BL"
+		(property "Footprint" "Circuits:SOIC-8_L4.9-W3.9-P1.27-LS6.0-BL"
 			(at 148.59 43.18 0)
 			(hide yes)
@@
 			)
 		)
-		(property "Footprint" "EasyEDA_Lib:USB-C-SMD_TYPE-C-16PIN-2MD-073"
+		(property "Footprint" "Circuits_Connectors:USB-C-SMD_TYPE-C-16PIN-2MD-073"
 			(at 35.56 40.64 0)
 			(hide yes)
@@
 			)
 		)
-		(property "Footprint" "Circuits:ESP32_S3_Supermini"
+		(property "Footprint" "Circuits_MCU:ESP32_S3_Supermini"
 			(at 38.1 135.89 0)
 			(show_name no)
@@
 			)
 		)
-		(property "Footprint" "Circuits:RJ45-TH_HC-WK88-H16-DB"
+		(property "Footprint" "Circuits_Connectors:RJ45-TH_HC-WK88-H16-DB"
 			(at 148.59 93.98 0)
 			(hide yes)
@@
 			)
 		)
-		(property "Footprint" "Connector_JST:JST_XH_S3B-XH-A_1x03_P2.50mm_Horizontal"
+		(property "Footprint" "Circuits_Connectors:CONN-TH_S3B-XH-A-LF-SN"
 			(at 102.87 143.51 0)
 			(hide yes)
