File: PCB/SensorBoard/HonkLockSensorBoard.kicad_sch (KiCad schematic)
At the start: 1 part

Commit message: Sensor board ready for mfg
Parts:
- added C1: 1uF, Capacitor_SMD:C_0805_2012Metric, symbol Device:C
- added C2, C3, C4: 0.1uF, Capacitor_SMD:C_0805_2012Metric, symbol Device:C
- added R1, R2: 10k, Resistor_SMD:R_0805_2012Metric, symbol PCM_SparkFun-Resistor:R
- added R6, R7: 33k, Resistor_SMD:R_0805_2012Metric, symbol PCM_SparkFun-Resistor:R
- added RJ1: (no value), Circuits:RJ45-TH_HC-WK88-H16-DB, symbol easyeda2:HC-WK88-H16-DB
- added TP1, TP2: TestPoint, PCM_SparkFun-Connector:TestPoint-1.25mm, symbol Connector:TestPoint
- added U2: (no value), Circuits:SOIC-8_L4.9-W3.9-P1.27-LS6.0-BL, symbol easyeda2:P82B715DR
Connections:
- net GND: now reaches U1.10 (N/C)
- net GND: now also U1.11 (A1), U1.12 (A0), U1.13 (VSS), U1.14 (N/C), U1.16 (N/C), U1.4 (N/C), U1.9 (N/C), C1.2, C2.2, C3.2, C4.1, RJ1.1, RJ1.10, RJ1.11 (+), RJ1.12 (-), RJ1.13 (+), RJ1.14 (-), RJ1.3, RJ1.5, RJ1.7, RJ1.8, RJ1.9, TP2.1, U2.4 (GND)
- net 3v3: now reaches U1.15 (VDD)
- net 3v3: now also C1.1, C2.1, C3.1, R6.2, R7.1, RJ1.4, TP1.1, U2.8 (VCC)
- net VDDIO: now reaches U1.2 (SENB/CS)
- net VDDIO: now also U1.8 (VDD_IO), C4.2, R1.1, R2.2
- net SensorSCL: now reaches U1.3 (SCL/SCLK)
- net SensorSCL: now also R1.2, R6.1, U2.6 (SY)
- net SensorSDA: now reaches U1.5 (SDA/MOSI)
- net SensorSDA: now also R2.1, R7.2, U2.3 (SX)
- new net ControllerSCL: RJ1.6, U2.7 (LY)
- new net ControllerSDA: RJ1.2, U2.2 (LX)
- no-connect marks 0 -> 5
Other:
- company: (none) -> tmuWolverine
- title: (none) -> HonkLock Tool Sensor
- moved on the sheet: U1

Commit message: sent to mfg
Parts:
- RJ1: footprint Circuits:RJ45-TH_HC-WK88-H16-DB -> Circuits_Connectors:RJ45-TH_HC-WK88-H16-DB
Changed lines of the file:
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@@
 			)
 		)
-		(property "Footprint" "Circuits:RJ45-TH_HC-WK88-H16-DB"
+		(property "Footprint" "Circuits_Connectors:RJ45-TH_HC-WK88-H16-DB"
 			(at 82.55 123.19 0)
 			(hide yes)
